Commit message: minor mass changes and more colour

File: description/robot_core.xacro (robot description, xacro)
@@ -37,5 +37,5 @@
       </geometry>
     </collision>
-    <xacro:inertial_box mass="0.5" x="0.2" y="0.2" z="0.1">
+    <xacro:inertial_box mass="1.0" x="0.2" y="0.2" z="0.1">
       <origin xyz="0.1 0 0.05" rpy="0 0 0"/>
     </xacro:inertial_box>
@@ -67,4 +67,5 @@
   </link>
   <gazebo reference="left_wheel">
+    <material>Gazebo/Blue</material>
   </gazebo>
   <!-- RIGHT WHEEL LINK -->
@@ -92,4 +93,5 @@
   </link>
   <gazebo reference="right_wheel">
+    <material>Gazebo/Blue</material>
   </gazebo>
   <!-- CASTER WHEEL LINK -->
@@ -111,11 +113,12 @@
       </geometry>
     </collision>
-    <xacro:inertial_sphere mass="0.1" radius="0.03">
+    <xacro:inertial_sphere mass="0.2" radius="0.03">
       <origin xyz="0 0 0" rpy="0 0 0"/>
     </xacro:inertial_sphere>
   </link>
   <gazebo reference="caster_wheel">
-    <mu1 value="0.001"/>
-    <mu2 value="0.001"/>
+    <material>Gazebo/Red</material>
+    <mu1 value="0.001" />
+    <mu2 value="0.001" />
   </gazebo>
 </robot>

Commit message: set up mapping

File: description/robot_core.xacro (robot description, xacro)
@@ -16,4 +16,12 @@
   <!-- BASE LINK -->
   <link name="base_link">
+  </link>
+  <!-- BASE FOOTPRINT LINK -->
+  <joint name="base_footprint_joint" type="fixed">
+    <parent link="base_link"/>
+    <child link="base_footprint"/>
+    <origin xyz="0 0 0" rpy="0 0 0"/>
+  </joint>
+  <link name="base_footprint">
   </link>
   <!-- CHASSIS LINK -->
