Commit message: flipped wheels

File: mole_ws/src/mole/description/robot_core.xacro (robot description, xacro)
@@ -55,6 +55,6 @@
     <parent link="base_link"/>
     <child link="left_wheel"/>
-    <origin xyz="0 0.115 0" rpy="-${pi/2} 0 0"/>
-    <axis xyz="0 0 1"/>
+    <origin xyz="0 -0.115 0" rpy="-${pi/2} 0 0"/>
+    <axis xyz="0 0 -1"/>
   </joint>
   <link name="left_wheel">
@@ -81,6 +81,6 @@
     <parent link="base_link"/>
     <child link="right_wheel"/>
-    <origin xyz="0 -0.115 0" rpy="${pi/2} 0 0"/>
-    <axis xyz="0 0 -1"/>
+    <origin xyz="0 0.115 0" rpy="${pi/2} 0 0"/>
+    <axis xyz="0 0 1"/>
   </joint>
   <link name="right_wheel">
