Commit message: more urdf changes

File: mole_ws/src/mole/description/lidar.xacro (robot description, xacro)
@@ -4,5 +4,5 @@
     <parent link="chassis"/>
     <child link="lidar"/>
-    <origin xyz="0.125 0 0.1" rpy="0 0 0"/>
+    <origin xyz="0.075 0 0.1" rpy="0 0 0"/>
   </joint>
   <link name="lidar">
@@ -18,5 +18,5 @@
       </geometry>
     </collision>
-    <xacro:inertial_cylinder mass="0.1" length="0.05" radius="0.04">
+    <xacro:inertial_cylinder mass="0.075" length="0.05" radius="0.04">
       <origin xyz="0 0 0" rpy="0 0 0"/>
     </xacro:inertial_cylinder>

File: mole_ws/src/mole/description/robot_core.xacro (robot description, xacro)
@@ -2,4 +2,16 @@
 <robot xmlns:xacro="http://www.ros.org/wiki/xacro">
   <xacro:include filename="inertial_macros.xacro"/>
+  <xacro:property name="chassis_length" value="0.2"/>
+  <xacro:property name="chassis_width" value="0.2"/>
+  <xacro:property name="chassis_height" value="0.1"/>
+  <xacro:property name="wheel_radius" value="0.03"/>
+  <xacro:property name="wheel_width" value="0.03"/>
+  <xacro:property name="wheel_mass" value="0.1"/>
+  <xacro:property name="wheel_offset_x" value="0.15"/>
+  <xacro:property name="wheel_offset_y" value="0.115"/>
+  <xacro:property name="wheel_offset_z" value="0.01"/>
+  <xacro:property name="caster_wheel_radius" value="0.03"/>
+  <xacro:property name="caster_wheel_mass" value="0.1"/>
+  <xacro:property name="caster_wheel_offset_x" value="0.05"/>
   <material name="white">
     <color rgba="1 1 1 1" />
@@ -29,22 +41,22 @@
     <parent link="base_link"/>
     <child link="chassis"/>
-    <origin xyz="-0.075 0 0"/>
+    <origin xyz="${-wheel_offset_x} 0 0" />
   </joint>
   <link name="chassis">
     <visual>
-      <origin xyz="0.1 0 0.05"/>
+      <origin xyz="${chassis_length/2} 0 ${chassis_height/2}"/>
       <geometry>
-        <box size="0.2 0.2 0.1"/>
+        <box size="${chassis_length} ${chassis_width} ${chassis_height}"/>
       </geometry>
       <material name="white"/>
     </visual>
     <collision>
-      <origin xyz="0.1 0 0.05"/>
+      <origin xyz="${chassis_length/2} 0 ${chassis_height/2}"/>
       <geometry>
-        <box size="0.2 0.2 0.1"/>
+        <box size="${chassis_length} ${chassis_width} ${chassis_height}"/>
       </geometry>
     </collision>
-    <xacro:inertial_box mass="1.0" x="0.2" y="0.2" z="0.1">
-      <origin xyz="0.1 0 0.05" rpy="0 0 0"/>
+    <xacro:inertial_box mass="1.0" x="${chassis_length} " y="${chassis_width}" z="${chassis_height}">
+      <origin xyz="${chassis_length/2} 0 ${chassis_height/2}" rpy="0 0 0"/>
     </xacro:inertial_box>
   </link>
@@ -55,11 +67,12 @@
     <parent link="base_link"/>
     <child link="left_wheel"/>
-    <origin xyz="0 -0.115 0" rpy="-${pi/2} 0 0"/>
-    <axis xyz="0 0 -1"/>
+    <origin xyz="0 ${wheel_offset_y} 0" rpy="-${pi/2} 0 0"/>
+    <axis xyz="0 0 1"/>
+    <dynamics damping="0.2" friction="0.1"/>
   </joint>
   <link name="left_wheel">
     <visual>
       <geometry>
-        <cylinder radius="0.03" length="0.03"/>
+        <cylinder radius="${wheel_radius}" length="${wheel_width}"/>
       </geometry>
       <material name="blue"/>
@@ -67,8 +80,8 @@
     <collision>
       <geometry>
-        <cylinder radius="0.03" length="0.03"/>
+        <cylinder radius="${wheel_radius}" length="${wheel_width}"/>
       </geometry>
     </collision>
-    <xacro:inertial_cylinder mass="0.1" length="0.03" radius="0.03">
+    <xacro:inertial_cylinder mass="${wheel_mass}" length="${wheel_width}" radius="${wheel_radius}">
       <origin xyz="0 0 0" rpy="0 0 0"/>
     </xacro:inertial_cylinder>
@@ -81,11 +94,12 @@
     <parent link="base_link"/>
     <child link="right_wheel"/>
-    <origin xyz="0 0.115 0" rpy="${pi/2} 0 0"/>
-    <axis xyz="0 0 1"/>
+    <origin xyz="0 ${-wheel_offset_y} 0" rpy="${pi/2} 0 0"/>
+    <axis xyz="0 0 -1"/>
+    <dynamics damping="0.2" friction="0.1"/>
   </joint>
   <link name="right_wheel">
     <visual>
       <geometry>
-        <cylinder radius="0.03" length="0.03"/>
+        <cylinder radius="${wheel_radius}" length="${wheel_width}"/>
       </geometry>
       <material name="blue"/>
@@ -93,8 +107,8 @@
     <collision>
       <geometry>
-        <cylinder radius="0.03" length="0.03"/>
+        <cylinder radius="${wheel_radius}" length="${wheel_width}"/>
       </geometry>
     </collision>
-    <xacro:inertial_cylinder mass="0.1" length="0.03" radius="0.03">
+    <xacro:inertial_cylinder mass="${wheel_mass}" length="${wheel_width}" radius="${wheel_radius}">
       <origin xyz="0 0 0" rpy="0 0 0"/>
     </xacro:inertial_cylinder>
@@ -107,10 +121,11 @@
     <parent link="chassis"/>
     <child link="caster_wheel"/>
-    <origin xyz="0.16 0 0"/>
+    <origin xyz="${caster_wheel_offset_x} 0 0"/>
+    <dynamics damping="0.2" friction="0.1"/>
   </joint>
   <link name="caster_wheel">
     <visual>
       <geometry>
-        <sphere radius="0.03"/>
+        <sphere radius="${caster_wheel_radius}"/>
       </geometry>
       <material name="red"/>
@@ -118,8 +133,8 @@
     <collision>
       <geometry>
-        <sphere radius="0.03"/>
+        <sphere radius="${caster_wheel_radius}"/>
       </geometry>
     </collision>
-    <xacro:inertial_sphere mass="0.2" radius="0.03">
+    <xacro:inertial_sphere mass="${caster_wheel_mass}" radius="${caster_wheel_radius}">
       <origin xyz="0 0 0" rpy="0 0 0"/>
     </xacro:inertial_sphere>
@@ -127,6 +142,6 @@
   <gazebo reference="caster_wheel">
     <material>Gazebo/Red</material>
-    <mu1 value="0.001" />
-    <mu2 value="0.001" />
+    <mu1 value="0.1" />
+    <mu2 value="0.1" />
   </gazebo>
 </robot>
